File: Nixie Clock.kicad_pcb (KiCad board)
At the start: 2 copper layers, 122.2 x 42.4 mm, 42 parts, among them J1 USB_C_Receptacle_USB2.0, Q1 FDS2672CT, Q26 MMBTA42, U1 ESP32-S2-WROVER, U1 UCC3803

Commit message: Finalized Bottom Plate with Gerbers
Parts:
- removed C10: 0.1uF 16v, Capacitors_SMD:C_0805
- removed C11: 1nF, Capacitors_SMD:C_0805
- removed C12: 0.1uF 250v, Capacitors_SMD:C_0805
- removed C14: 47uF 16v, Capacitors_SMD:C_1210
- removed C15: 560pF 250v, Capacitors_SMD:C_0603
- removed C16, C9: 100uF 16v, Capacitors_SMD:C_1210
- removed C18: 0.1uF, Capacitors_SMD:C_0805
- removed C7: 430pF, Capacitors_SMD:C_0805
- removed G***: LOGO, Symbol:copyright
- removed G***: OSHW_logo_silkscreen-front_5mm, NixieSupply5vto170vDCMBoostMini_socket:OSHW_logo_silkscreen-front_5mm
- removed L2, L5: 60ohm 100Mhz, Resistors_SMD:R_0805
- removed L3: 33uH, NixieSupply5vto160vDCMBoost_socket:Choke_SMD_12x12mm_Wurth_WE-PD
- removed N1, N2, N3, N4: IN-16, nixies-us:nixies-us-IN-16
- removed Q26: MMBTA42, TO_SOT_Packages_SMD:SOT-23
- removed R10: 0.1 1/2W, Resistors_SMD:R_0805
- removed R12: 4.12k, Resistors_SMD:R_0805
- removed R15: 634k, Resistors_SMD:R_0805
- removed R16: 7.68k, Resistors_SMD:R_0805
- removed R7: 2k, Resistors_SMD:R_0805
- removed R8: 1k, Resistors_SMD:R_0805
- removed R9: 100k, Resistors_SMD:R_0805
- removed the U1 at (136.1, 54.5)
- removed the U1 at (237.5, 69.3)
- added C4: 100n, Capacitor_SMD:C_0402_1005Metric, B.Cu at (136.6, 73.3)
- added D3: ~, LED_SMD:LED_WS2812B-2020_PLCC4_2.0x2.0mm, F.Cu at (167.6, 83.8)
- added D4: ~, LED_SMD:LED_WS2812B-2020_PLCC4_2.0x2.0mm, F.Cu at (188.0, 83.8)
- added D5: ~, LED_SMD:LED_WS2812B-2020_PLCC4_2.0x2.0mm, F.Cu at (203.2, 83.8)
- added J2: Debug, Connector_PinHeader_2.54mm:PinHeader_1x04_P2.54mm_Vertical, F.Cu at (138.8, 99.9)
- added J3: Conn_01x23_Pin, Connector_PinSocket_2.54mm:PinSocket_1x23_P2.54mm_Vertical, F.Cu at (205.7, 62.5)
- added J4: Conn_01x23_Pin, Connector_PinSocket_2.54mm:PinSocket_1x23_P2.54mm_Vertical, F.Cu at (149.9, 105.2)
- added PD1: BH1730, Sensor_Ambient:WSOF6, B.Cu at (140.5, 63.2)
- added Q2: NMOS_GSD, Package_TO_SOT_SMD:SOT-23, B.Cu at (180.3, 95.5)
- added SW1: SW_Push, Button_Switch_SMD:SW_SPST_SKQG_WithStem, F.Cu at (141.1, 73.8)
- added SW2: SW_Push, Button_Switch_SMD:SW_SPST_SKQG_WithStem, F.Cu at (141.1, 93.9)
- added U1: 74141, Package_DIP:DIP-16_W7.62mm, F.Cu at (158.8, 74.9)
- added U2: 74141, Package_DIP:DIP-16_W7.62mm, F.Cu at (184.2, 74.9)
- added U3: 74141, Package_DIP:DIP-16_W7.62mm, F.Cu at (176.5, 92.7)
- added U4: 74141, Package_DIP:DIP-16_W7.62mm, F.Cu at (201.9, 92.7)
- added U5: ESP32-S2-Solo, RF_Module:ESP32-S3-WROOM-1, B.Cu at (141.7, 83.8)
- added U6: AMS1117-3.3, Package_TO_SOT_SMD:SOT-223-3_TabPin2, B.Cu at (214.9, 98.3)
- added U7: ~, omnixie:8200HV, F.Cu at (216.7, 84.1)
- C1, C2: value 1uF 250v -> 10u; footprint Capacitors_SMD:C_1812_HandSoldering -> Capacitor_SMD:C_0603_1608Metric; moved to B.Cu
- C3: value 0.1uF 250v -> 10u; footprint Capacitors_SMD:C_0805 -> Capacitor_SMD:C_0603_1608Metric; moved to B.Cu
- C5: value 220pF -> 100n; footprint Capacitors_SMD:C_0805 -> Capacitor_SMD:C_0402_1005Metric; moved to B.Cu
- C6: value 100pF 250v -> 100n; footprint Capacitors_SMD:C_0805 -> Capacitor_SMD:C_0402_1005Metric; moved to B.Cu
- D1: value ES1D -> PRTR5V0U2X; footprint Diodes_SMD:D_SMA -> Package_TO_SOT_SMD:SOT-143; moved to B.Cu
- D2: value BAT54 -> ~; footprint Diodes_SMD:D_SOD-323_HandSoldering -> LED_SMD:LED_WS2812B-2020_PLCC4_2.0x2.0mm
- J1: value USB_C_Receptacle_USB2.0 -> Type-C 31-M-12; moved to B.Cu
- Q1: value FDS2672CT -> NMOS_GSD; footprint etaclock:SOIC-8-N -> Package_TO_SOT_SMD:SOT-23; moved to B.Cu
- R1: value 1k -> 5k1; footprint Resistors_SMD:R_0805 -> Resistor_SMD:R_0402_1005Metric; moved to B.Cu
- R2: value 60.4k -> 5k1; footprint Resistors_SMD:R_0805 -> Resistor_SMD:R_0402_1005Metric; moved to B.Cu
- R3: value N.U. -> 10k; footprint Resistors_SMD:R_0805 -> Resistor_SMD:R_0402_1005Metric; moved to B.Cu
- R4: value 100k -> TBD; footprint Resistors_SMD:R_0805 -> Resistor_SMD:R_0603_1608Metric_Pad0.98x0.95mm_HandSolder; moved to B.Cu
- R5: value 0 Ohm -> TBD; footprint Resistors_SMD:R_0805 -> Resistor_SMD:R_0603_1608Metric_Pad0.98x0.95mm_HandSolder; moved to B.Cu
- moved C3 120.0 mm to (137.1, 71.8), turned to 180 degrees
- moved C6 113.7 mm to (138.4, 64.5), turned to 120 degrees
- moved R3 99.0 mm to (138.7, 73.3)
- moved C5 93.7 mm to (139.7, 71.8)
- moved D2 83.1 mm to (152.4, 83.8), turned to 180 degrees
- moved R5 67.4 mm to (180.3, 100.6), turned to 90 degrees
- moved J1 58.3 mm to (225.8, 83.8), turned to -90 degrees
- moved C2 51.6 mm to (209.5, 99.3), turned to -90 degrees
- moved C1 48.6 mm to (208.7, 95.8), turned to 180 degrees
- moved Q1 40.1 mm to (204.9, 71.1), turned to 0 degrees
- moved D1 30.6 mm to (215.4, 83.8), turned to 90 degrees
- moved R1 29.9 mm to (219.5, 82.3), turned to 180 degrees
- moved R4 22.8 mm to (205.2, 67.1)
- moved R2 21.8 mm to (219.5, 85.3), turned to 180 degrees
Connections:
- C1 pad 1: (no net) -> +5V
- C1 pad 2: (no net) -> GND
- C2 pad 1: (no net) -> +3V3
- C2 pad 2: (no net) -> GND
- C3 pad 1: (no net) -> +3V3
- C3 pad 2: (no net) -> GND
- C5 pad 1: (no net) -> RST
- C5 pad 2: (no net) -> GND
- C6 pad 1: (no net) -> +3V3
- C6 pad 2: (no net) -> GND
- D1 pad 1: (no net) -> GND
- D1 pad 2: (no net) -> D+
- D2 pad 1: (no net) -> Net-(D2-DOUT)
- D2 pad 2: (no net) -> GND
- J1 pad A1: Net-(J1-GND-PadA1) -> GND
- J1 pad A12: Net-(J1-GND-PadA1) -> GND
- J1 pad A4: Net-(J1-VBUS-PadA4) -> +5V
- J1 pad A5: unconnected-(J1-CC1-PadA5) -> Net-(J1-CC1)
- J1 pad A6: unconnected-(J1-D+-PadA6) -> D+
- J1 pad A7: unconnected-(J1-D--PadA7) -> D-
- J1 pad A9: Net-(J1-VBUS-PadA4) -> +5V
- J1 pad B1: Net-(J1-GND-PadA1) -> GND
- J1 pad B12: Net-(J1-GND-PadA1) -> GND
- J1 pad B4: Net-(J1-VBUS-PadA4) -> +5V
- J1 pad B5: unconnected-(J1-CC2-PadB5) -> Net-(J1-CC2)
- J1 pad B6: unconnected-(J1-D+-PadB6) -> D+
- J1 pad B7: unconnected-(J1-D--PadB7) -> D-
- J1 pad B9: Net-(J1-VBUS-PadA4) -> +5V
- J1 pad S1: unconnected-(J1-SHIELD-PadS1) -> GND
- Q1 pad 1: (no net) -> C_RDP
- Q1 pad 2: (no net) -> GND
- Q1 pad 3: (no net) -> Net-(Q1-D)
- R1 pad 1: (no net) -> Net-(J1-CC1)
- R1 pad 2: (no net) -> GND
- R2 pad 1: (no net) -> Net-(J1-CC2)
- R2 pad 2: (no net) -> GND
- R3 pad 1: (no net) -> RST
- R3 pad 2: (no net) -> +3V3
- R4 pad 1: (no net) -> RDP
- R4 pad 2: (no net) -> Net-(Q1-D)
- R5 pad 1: (no net) -> LDP
- R5 pad 2: (no net) -> Net-(Q2-D)
Routing:
- net (no net): track 361.3 -> 0.00 mm, vias 32 -> 0
- net +5V: track 0.00 -> 144.4 mm, vias 0 -> 3
- net +3V3: track 0.00 -> 138.5 mm, vias 0 -> 6
- net D+: track 0.00 -> 81.0 mm, vias 0 -> 2
- net D-: track 0.00 -> 80.4 mm, vias 0 -> 2
- net C_RDP: track 0.00 -> 52.1 mm
- net 2_C: track 0.00 -> 48.6 mm
- net 4_A: track 0.00 -> 46.0 mm
- net 2_B: track 0.00 -> 45.5 mm
- net 4_D: track 0.00 -> 43.4 mm
- net 2_D: track 0.00 -> 39.9 mm
- net 4_B: track 0.00 -> 37.4 mm
- net 2_A: track 0.00 -> 36.9 mm
- net 4_C: track 0.00 -> 34.3 mm
- net 1_C: track 0.00 -> 32.2 mm
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- added copper zone on B.Cu, net GND
- added copper zone on F.Cu, net GND
- added copper zone on In1.Cu, net GND
- added copper zone on In2.Cu, net GND
- removed copper zone on B.Cu, net (none)
- removed copper zone on F.Cu, net (none)
Other:
- board size 122.2 x 42.4 mm -> 101.6 x 50.8 mm
- copper layers 2 -> 4
- board text added: "3v3"
- board text added: "BOOT"
- board text added: "GND"
- board text added: "RST"
- board text added: "RX"
- board text added: "TX"
- board text removed: "Mark Smith 2018"
- board text removed: "NixieSupplyMini Rev3_1812"
- board text removed: "www.surfncircuits.com"
